File: Z_Brake/Z_Brake.sch (KiCad schematic (older format))
At the start: 26 parts, among them K1 EC2-24NU, K2 EC2-24NU, P1 CONN_01X04, P2 CONN_01X02, P3 CONN_01X04, Q1 2N7002, U1 LM397

Commit message: Final PCB
Connections:
- net VDD: now also D4.2 (A); no longer D4.1 (K)
- net at R7.1: now also D4.1 (K); no longer D4.2 (A)
Other:
- moved on the sheet: D4
Changed lines of the file:
@@
 Connection ~ 1750 3100
-$Comp
-L Device:LED_ALT D4
-U 1 1 5A282358
-P 6500 4450
-F 0 "D4" V 6500 4600 50  0000 C CNN
-F 1 "LED" V 6500 4250 50  0000 C CNN
-F 2 "LED_SMD:LED_0603_1608Metric_Pad1.05x0.95mm_HandSolder" H 6500 4450 50  0001 C CNN
-F 3 "" H 6500 4450 50  0000 C CNN
-F 4 "160-1184-1-ND" V 6500 4450 50  0001 C CNN "DKPN"
-	1    6500 4450
-	0    1    1    0
-$EndComp
 $Comp
 L Device:R R7
@@
 	1    0    0    -1
 $EndComp
+$Comp
+L Device:LED_ALT D4
+U 1 1 5A282358
+P 6500 4450
+F 0 "D4" V 6500 4600 50  0000 C CNN
+F 1 "LED" V 6500 4250 50  0000 C CNN
+F 2 "LED_SMD:LED_0603_1608Metric_Pad1.05x0.95mm_HandSolder" H 6500 4450 50  0001 C CNN
+F 3 "" H 6500 4450 50  0000 C CNN
+F 4 "160-1184-1-ND" V 6500 4450 50  0001 C CNN "DKPN"
+	1    6500 4450
+	0    -1   -1   0
+$EndComp
 $EndSCHEMATC

Commit message: Add fab files
Parts:
- C1: MPN (none) -> CL10B224KB8VPNC; Manufacturer (none) -> Samsung
- D1: AO Part Number PC-MS0056 -> (none); MPN (none) -> SMAZ10-13-F; Manufacturer (none) -> Diodes Incorporated; Part Number SMAZ10-13-F -> (none)
- D2, D3: MPN (none) -> BAT48ZFILM; Manufacturer (none) -> STMicroelectronics; Part Number BAT48ZFILM -> (none)
- D4: MPN (none) -> LTST-C190YKT; Manufacturer (none) -> Lite-On Inc.
- D5: MPN (none) -> CDBA340-HF; Manufacturer (none) -> Comchip Technology; Part Number CDBA340-HF -> (none)
- K1, K2: MPN (none) -> EC2-24NU; Manufacturer (none) -> Kemet; Part Number EC2-24NU -> (none)
- P1, P3: MPN (none) -> 0705430003; Manufacturer (none) -> Molex
- P2: MPN (none) -> 0705430001; Manufacturer (none) -> Molex
- Q1: MPN (none) -> 2N7002 TR PBFREE; Manufacturer (none) -> Central Semiconductor Corp
- R1: MPN (none) -> RC0603FR-0712K4L; Manufacturer (none) -> YAGEO
- R2, R3, R5, R6: MPN (none) -> RC0603FR-0710KL; Manufacturer (none) -> YAGEO
- R4: MPN (none) -> RC0603FR-07180KL; Manufacturer (none) -> YAGEO
- R7: MPN (none) -> RC0603FR-073K3L; Manufacturer (none) -> YAGEO
- RV1, RV2: MPN (none) -> AVR-M2012C390KT6AB; Manufacturer (none) -> TDK
- U1: MPN (none) -> LM397MF/NOPB; Manufacturer (none) -> TI
Other:
- note added: "1.0.0"
- note added: "Latest Edit 09-10-2021"
- note added: "v1.0.0 - Original conversion to \nsingle motor output"
- note removed: "C"
- note removed: "Latest Edit 09-14-2018"
- note removed: "REV. A Original Design"
- note removed: "REV. B Relays moved on PCB design\nto allow space for 4-Pin motor\nconnectors."
- note removed: "REV. C Varistors added to motor\nwinding connectors to suppress\nvoltage spikes when relays\ndisconnect motor windings. PCB\nchanged to add varistors."
Changed lines of the file:
@@
 F 3 "" H 3450 4400 50  0000 C CNN
 F 4 "1276-6600-1-ND" V 3450 4400 50  0001 C CNN "DKPN"
+F 5 "CL10B224KB8VPNC" V 3450 4400 50  0001 C CNN "MPN"
+F 6 "Samsung" V 3450 4400 50  0001 C CNN "Manufacturer"
 	1    3450 4400
 	0    1    1    0
@@
 F 2 "Diode_SMD:D_SMA_Handsoldering" H 2500 6150 50  0001 C CNN
 F 3 "" H 2500 6150 50  0000 C CNN
-F 4 "SMAZ10-13-F" H 2500 6150 60  0001 C CNN "Part Number"
+F 4 "SMAZ10-13-F" H 2500 6150 60  0001 C CNN "MPN"
 F 5 "Digikey" H 2500 6150 60  0001 C CNN "Primary Supplier"
 F 6 "SMAZ10-FDICT-ND" H 2500 6150 60  0001 C CNN "DKPN"
-F 7 "PC-MS0056" H 2500 6150 60  0001 C CNN "AO Part Number"
+F 7 "Diodes Incorporated" V 2500 6150 50  0001 C CNN "Manufacturer"
 	1    2500 6150
 	0    1    1    0
@@
 F 3 "" H 1400 1900 50  0000 C CNN
 F 4 "WM4802-ND" H 1400 1900 50  0001 C CNN "DKPN"
+F 5 "Molex" H 1400 1900 50  0001 C CNN "Manufacturer"
+F 6 "0705430003" H 1400 1900 50  0001 C CNN "MPN"
 	1    1400 1900
 	-1   0    0    -1
@@
 F 3 "" H 8700 1900 50  0000 C CNN
 F 4 "WM4802-ND" H 8700 1900 50  0001 C CNN "DKPN"
+F 5 "0705430003" H 8700 1900 50  0001 C CNN "MPN"
+F 6 "Molex" H 8700 1900 50  0001 C CNN "Manufacturer"
 	1    8700 1900
 	1    0    0    -1
@@
 F 2 "Diode_SMD:D_SOD-123" H 5300 1950 50  0001 C CNN
 F 3 "" H 5300 1950 50  0000 C CNN
-F 4 "BAT48ZFILM" H 5300 1950 60  0001 C CNN "Part Number"
+F 4 "BAT48ZFILM" H 5300 1950 60  0001 C CNN "MPN"
 F 5 "Digikey" H 5300 1950 60  0001 C CNN "Primary Supplier"
 F 6 "497-5712-1-ND" H 5300 1950 60  0001 C CNN "DKPN"
+F 7 "STMicroelectronics" V 5300 1950 50  0001 C CNN "Manufacturer"
 	1    5300 1950
 	0    1    1    0
@@
 F 2 "Diode_SMD:D_SOD-123" H 5300 3250 50  0001 C CNN
 F 3 "" H 5300 3250 50  0000 C CNN
-F 4 "BAT48ZFILM" H 5300 3250 60  0001 C CNN "Part Number"
+F 4 "BAT48ZFILM" H 5300 3250 60  0001 C CNN "MPN"
 F 5 "Digikey" H 5300 3250 60  0001 C CNN "Primary Supplier"
 F 6 "497-5712-1-ND" H 5300 3250 60  0001 C CNN "DKPN"
+F 7 "STMicroelectronics" V 5300 3250 50  0001 C CNN "Manufacturer"
 	1    5300 3250
 	0    1    1    0
@@
 F 3 "" H 1400 3200 50  0000 C CNN
 F 4 "WM4800-ND" H 1400 3200 50  0001 C CNN "DKPN"
+F 5 "Molex" H 1400 3200 50  0001 C CNN "Manufacturer"
+F 6 "0705430001" H 1400 3200 50  0001 C CNN "MPN"
 	1    1400 3200
 	-1   0    0    1
@@
 F 3 "" H 6500 4850 50  0000 C CNN
 F 4 "311-3.30KHRCT-ND" H 6500 4850 50  0001 C CNN "DKPN"
+F 5 "RC0603FR-073K3L" H 6500 4850 50  0001 C CNN "MPN"
+F 6 "YAGEO" H 6500 4850 50  0001 C CNN "Manufacturer"
 	1    6500 4850
 	1    0    0    -1
@@
 F 3 "" H 4850 5500 50  0000 C CNN
 F 4 "311-10.0KHRCT-ND" V 4850 5500 50  0001 C CNN "DKPN"
+F 5 "RC0603FR-0710KL" V 4850 5500 50  0001 C CNN "MPN"
+F 6 "YAGEO" V 4850 5500 50  0001 C CNN "Manufacturer"
 	1    4850 5500
 	0    1    1    0
@@
 F 3 "" H 3450 4700 50  0001 C CNN
 F 4 "311-180KHRCT-ND" V 3450 4700 50  0001 C CNN "DKPN"
+F 5 "RC0603FR-07180KL" V 3450 4700 50  0001 C CNN "MPN"
+F 6 "YAGEO" V 3450 4700 50  0001 C CNN "Manufacturer"
 	1    3450 4700
 	0    1    1    0
@@
 F 3 "" H 2500 5050 50  0000 C CNN
 F 4 "311-10.0KHRCT-ND" H 2500 5050 50  0001 C CNN "DKPN"
+F 5 "RC0603FR-0710KL" H 2500 5050 50  0001 C CNN "MPN"
+F 6 "YAGEO" H 2500 5050 50  0001 C CNN "Manufacturer"
 	1    2500 5050
 	1    0    0    -1
@@
 F 3 "" H 1900 5050 50  0000 C CNN
 F 4 "311-12.4KHRCT-ND" H 1900 5050 50  0001 C CNN "DKPN"
+F 5 "RC0603FR-0712K4L" H 1900 5050 50  0001 C CNN "MPN"
+F 6 "YAGEO" H 1900 5050 50  0001 C CNN "Manufacturer"
 	1    1900 5050
 	1    0    0    -1
@@
 F 3 "" H 1900 6150 50  0000 C CNN
 F 4 "311-10.0KHRCT-ND" H 1900 6150 50  0001 C CNN "DKPN"
+F 5 "RC0603FR-0710KL" H 1900 6150 50  0001 C CNN "MPN"
+F 6 "YAGEO" H 1900 6150 50  0001 C CNN "Manufacturer"
 	1    1900 6150
 	1    0    0    -1
@@
 F 3 "" H 4400 4950 50  0000 C CNN
 F 4 "311-10.0KHRCT-ND" H 4400 4950 50  0001 C CNN "DKPN"
+F 5 "RC0603FR-0710KL" H 4400 4950 50  0001 C CNN "MPN"
+F 6 "YAGEO" H 4400 4950 50  0001 C CNN "Manufacturer"
 	1    4400 4950
 	1    0    0    -1
@@
 F 2 "Diode_SMD:D_SMA_Handsoldering" H 2400 3100 50  0001 C CNN
 F 3 "" H 2400 3100 50  0000 C CNN
-F 4 "CDBA340-HF" H 2400 3100 60  0001 C CNN "Part Number"
+F 4 "CDBA340-HF" H 2400 3100 60  0001 C CNN "MPN"
 F 5 "Digikey" H 2400 3100 60  0001 C CNN "Primary Supplier"
 F 6 "641-1748-1-ND" H 2400 3100 60  0001 C CNN "DKPN"
+F 7 "Comchip Technology" H 2400 3100 50  0001 C CNN "Manufacturer"
 	1    2400 3100
 	-1   0    0    1
@@
 F 3 "" H 8000 1550 50  0000 C CNN
 F 4 "445-2549-1-ND" H 8000 1550 50  0001 C CNN "DKPN"
+F 5 "AVR-M2012C390KT6AB" H 8000 1550 50  0001 C CNN "MPN"
+F 6 "TDK" H 8000 1550 50  0001 C CNN "Manufacturer"
 	1    8000 1550
 	1    0    0    -1
@@
 F 3 "" H 8000 2350 50  0000 C CNN
 F 4 "445-2549-1-ND" H 8000 2350 50  0001 C CNN "DKPN"
+F 5 "AVR-M2012C390KT6AB" H 8000 2350 50  0001 C CNN "MPN"
+F 6 "TDK" H 8000 2350 50  0001 C CNN "Manufacturer"
 	1    8000 2350
 	1    0    0    -1
@@
 Z_Brake.sch
 Text Notes 8150 7650 0    59   ~ 0
-Latest Edit 09-14-2018
+Latest Edit 09-10-2021
 Text Notes 9200 950  0    118  ~ 0
 REVISION HISTORY
-Text Notes 9250 1150 0    59   ~ 0
-REV. A Original Design
-Text Notes 9250 1500 0    59   ~ 0
-REV. B Relays moved on PCB design\nto allow space for 4-Pin motor\nconnectors.
-Text Notes 9250 2050 0    59   ~ 0
-REV. C Varistors added to motor\nwinding connectors to suppress\nvoltage spikes when relays\ndisconnect motor windings.  PCB\nchanged to add varistors.
 Text Notes 2800 6850 0    59   ~ 0
 Approx. 22.7 VDC
@@
 USE - This board prevents the print head\nassembly from falling when power is\ndisconnected.
 Text Notes 10600 7650 0    59   ~ 0
-C
+1.0.0
 Wire Wire Line
 	5300 2200 5550 2200
@@
 F 3 "" H 5450 5500 50  0000 L CNN
 F 4 "1514-2N7002TRPBFREECT-ND" H 5450 5500 50  0001 C CNN "DKPN"
+F 5 "2N7002 TR PBFREE" H 5450 5500 50  0001 C CNN "MPN"
+F 6 "Central Semiconductor Corp" H 5450 5500 50  0001 C CNN "Manufacturer"
 	1    5450 5500
 	1    0    0    -1
@@
 F 3 "" H 3500 5500 60  0001 C CNN
 F 4 "LM397MF/NOPBCT-ND" H 3450 5500 50  0001 C CNN "DKPN"
+F 5 "LM397MF/NOPB" H 3450 5500 50  0001 C CNN "MPN"
+F 6 "TI" H 3450 5500 50  0001 C CNN "Manufacturer"
 	1    3450 5500
 	1    0    0    -1
@@
 F 2 "ec2:EC2_Relay" H 4200 1450 60  0001 C CNN
 F 3 "" H 4200 1450 60  0001 C CNN
-F 4 "EC2-24NU" H 4450 1950 60  0001 C CNN "Part Number"
+F 4 "EC2-24NU" H 4450 1950 60  0001 C CNN "MPN"
 F 5 "Digikey" H 4450 1950 60  0001 C CNN "Primary Supplier"
 F 6 "399-11037-5-ND" H 4450 1950 60  0001 C CNN "DKPN"
+F 7 "Kemet" H 4450 1950 50  0001 C CNN "Manufacturer"
 	1    4450 1950
 	1    0    0    -1
@@
 F 2 "ec2:EC2_Relay" H 4200 2750 60  0001 C CNN
 F 3 "" H 4200 2750 60  0001 C CNN
-F 4 "EC2-24NU" H 4450 3250 60  0001 C CNN "Part Number"
+F 4 "EC2-24NU" H 4450 3250 60  0001 C CNN "MPN"
 F 5 "Digikey" H 4450 3250 60  0001 C CNN "Primary Supplier"
 F 6 "399-11037-5-ND" H 4450 3250 60  0001 C CNN "DKPN"
+F 7 "Kemet" H 4450 3250 50  0001 C CNN "Manufacturer"
 	1    4450 3250
 	1    0    0    -1
@@
 F 3 "" H 6500 4450 50  0000 C CNN
 F 4 "160-1184-1-ND" V 6500 4450 50  0001 C CNN "DKPN"
+F 5 "LTST-C190YKT" V 6500 4450 50  0001 C CNN "MPN"
+F 6 "Lite-On Inc." V 6500 4450 50  0001 C CNN "Manufacturer"
 	1    6500 4450
 	0    -1   -1   0
 $EndComp
+Text Notes 9250 1150 0    59   ~ 0
+v1.0.0 - Original conversion to \nsingle motor output
 $EndSCHEMATC
