File: Z_Brake_SMD_Relay/Z_Brake.kicad_pcb (KiCad board)
At the start: 2 copper layers, 47 x 47 mm, 28 parts, among them K1 EC2-24NU, K2 EC2-24NU, P1 CONN_01X04, P2 CONN_01X02, P3 CONN_01X04, Q1 2N7002, U1 LM397

Commit message: Added smt relay version
Parts:
- K1, K2: footprint ec2:EC2_Relay -> Relay_SMD:Relay_DPDT_Kemet_EE2_NU
- moved K1 1.55 mm to (94.9, 95.2), turned to 180 degrees
- moved K2 1.53 mm to (83.0, 95.2), turned to 180 degrees
Routing:
- net Net-(D2-Pad2): track 31.5 -> 26.9 mm
- net Net-(K2-Pad4): track 31.3 -> 33.9 mm, vias 0 -> 1
- net Net-(K1-Pad9): track 31.3 -> 33.8 mm, vias 0 -> 1
- net VDD: track 72.8 -> 70.5 mm
- net Net-(K2-Pad10): track 5.08 -> 7.29 mm
- net Net-(K1-Pad10): track 5.08 -> 7.29 mm
- net Net-(K2-Pad9): track 32.9 -> 34.4 mm, vias 0 -> 1
- net Net-(K1-Pad4): track 32.9 -> 34.1 mm, vias 0 -> 1
- net Net-(K2-Pad8): track 9.07 -> 9.88 mm
- net Net-(K1-Pad5): track 9.15 -> 9.90 mm
